Commit message: added efford control

File: src/z1_model/urdf/gazebo.xacro (robot description, xacro)
@@ -1,47 +1,36 @@
 <?xml version="1.0"?>
 <robot xmlns:xacro="http://www.ros.org/wiki/xacro">
-    <xacro:macro name="joint_controller" params="name">
+    <xacro:macro name="joint_controller" params="name initial_position">
         <joint name="${name}">
             <command_interface name="effort">
-            <param name="min">-33</param>
-            <param name="max">33</param>
+                <param name="min">-33</param>
+                <param name="max">33</param>
             </command_interface>
-            <state_interface name="position"/>
+            <!-- <state_interface name="position"/> -->
+            <state_interface name="position">
+                <param name="initial_value">${initial_position}</param>    <!-- начальный угол, рад -->
+            </state_interface>
             <state_interface name="velocity"/>
             <state_interface name="effort"/>
         </joint>
     </xacro:macro>
-    <!-- <gazebo>
-        <plugin name="gazebo_ros_control" filename="libgazebo_ros_control.so">
-            <robotNamespace>/z1_gazebo</robotNamespace>
-            <robotSimType>gazebo_ros_control/DefaultRobotHWSim</robotSimType>
-        </plugin>
-    </gazebo> -->
-    <plugin name="gazebo_ros_control" filename="libgazebo_ros_control.so">
-        <robotNamespace>/z1</robotNamespace>
-    </plugin>
     <ros2_control name="Z1GazeboSystem" type="system">
         <hardware>
             <plugin>gz_ros2_control/GazeboSimSystem</plugin>
         </hardware>
-        <xacro:joint_controller name="joint1"/>
-        <xacro:joint_controller name="joint2"/>
-        <xacro:joint_controller name="joint3"/>
-        <xacro:joint_controller name="joint4"/>
-        <xacro:joint_controller name="joint5"/>
-        <xacro:joint_controller name="joint6"/>
+        <xacro:joint_controller name="joint1" initial_position="0.0"/>
+        <xacro:joint_controller name="joint2" initial_position="0.0"/>
+        <xacro:joint_controller name="joint3" initial_position="-0.035"/> <!-- примерно 2 градуса -->
+        <xacro:joint_controller name="joint4" initial_position="-1.047"/> <!-- примерно 60 градусов -->
+        <xacro:joint_controller name="joint5" initial_position="0.0"/>
+        <xacro:joint_controller name="joint6" initial_position="0.0"/>
     </ros2_control>
-    <plugin filename="libgz_ros2_control-system.so"
-            name="gz_ros2_control::GazeboSimROS2ControlPlugin">
-        <parameters>$(find z1_model)/config/z1_controllers.yaml</parameters>
-    </plugin>
-    <!-- <gazebo reference="link04">
-        <self_collide>true</self_collide>
+    <gazebo>
+        <plugin name="gz_ros2_control::GazeboSimROS2ControlPlugin" filename="gz_ros2_control-system"> <!-- lib .so -->
+            <parameters>$(find z1_model)/config/z1_controllers.yaml</parameters>
+            <ros>
+                <namespace>/z1</namespace>
+            </ros>
+        </plugin>
     </gazebo>
-    <gazebo reference="link05">
-        <self_collide>true</self_collide>
-    </gazebo>
-    <gazebo reference="link06">
-        <self_collide>true</self_collide>
-    </gazebo> -->
 </robot>
