Commit message: removed unnecessary comments

File: src/entrance_group_v3/urdf/button_macro.xacro (robot description, xacro)
@@ -3,31 +3,6 @@
   Xacro-макрос одной кнопки домофона.
   Каждая кнопка состоит из ДВУХ звеньев:
-    * button_<idx>      - тело кнопки (серый пластик, квадратный box).
-                          Двигается prismatic-шарниром вглубь домофона.
-    * button_<idx>_cap  - тонкая накладка с цифрой/символом, жёстко прикреплённая
-                          к лицевой стороне кнопки. Текстура нанесена только сюда,
-                          поэтому никакие боковые грани кнопки не получают цифру.
-  Также генерируются:
-    * button_<idx>_joint  - prismatic, ход 0...3 мм, пружинный возврат.
-    * <gazebo> блок для пружины этого шарнира.
-    * <gazebo> блок с PBR-материалом для накладки (текстура с цифрой).
-    * <gazebo> блок с PBR-материалом для тела кнопки (общая пластиковая текстура).
-  Параметры:
-    idx          - числовой индекс кнопки (1..12) - попадает в имена звеньев.
-    label_name   - человекочитаемое имя для текстуры: "1".."9", "0", "star", "hash".
-                   Используется как basename для файла:
-                   model://entrance_group_v3/materials/textures/button_<label_name>.png
-    parent       - имя parent-звена (intercom_body).
-    xyz          - позиция тела кнопки в системе parent (string "x y z").
-    bx, by, bz   - размер тела кнопки по осям X/Y/Z, в метрах
-                   (по умолчанию 8x10x10 мм: bx = глубина внутрь домофона, by/bz = фасад).
-                   Разделены на 3 параметра вместо одной строки "x y z",
-                   чтобы файл был совместим с JS-парсерами xacro
-                   (URDF Visualiser в VS Code и др.), которые не поддерживают
-                   Python-методы строк (.split() и др.).
-    cap_thickness - толщина накладки (по умолчанию 0.5 мм).
-    travel       - максимальный ход кнопки в м (по умолчанию 0.003 = 3 мм).
-    spring_k     - жёсткость возвратной пружины Н/м (по умолчанию 500).
-    damping      - демпфирование шарнира (по умолчанию 3.0).
+    * button_${button_name}      - тело кнопки (серый пластик, квадратный box). Двигается prismatic-шарниром вглубь домофона.
+    * button_${button_name}_cap  - тонкая накладка с цифрой/символом, жёстко прикреплённая к лицевой стороне кнопки. Текстура нанесена только сюда
 -->
 <robot xmlns:xacro="http://www.ros.org/wiki/xacro">
@@ -47,7 +22,4 @@
         <geometry>
           <box size="${bx} ${by} ${bz}"/>
-          <!-- <mesh filename="package://entrance_group_v3/materials/button_0.obj" scale="1.0 1.0 1.0"/> -->
-          <!-- <mesh filename="../materials/button_0.obj" scale="1.0 1.0 1.0"/> -->
-          <!-- <mesh filename="$(find entrance_group_v3)/materials/button_0.obj" scale="1.0 1.0 1.0"/> -->
         </geometry>
         <material name="button_${button_name}_body_mat">
@@ -124,4 +96,5 @@
               rpy="0 0 0"/>
     </joint>
+    <!-- gazebo-разделитель, чтобы текстура родителя не переходила на дочерние fixed-элементы -->
     <gazebo reference="button_${button_name}_cap_fixed">
       <preserveFixedJoint>true</preserveFixedJoint>
@@ -142,5 +115,4 @@
         </material>
       </visual>
-      <!-- <visual><material><pbr><metal><albedo_map>model://entrance_group_v3/materials/textures/button_1.png</albedo_map><metalness>0.0</metalness><roughness>0.4</roughness></metal></pbr></material></visual> -->
     </gazebo>
     <!-- ====== 5. PBR-материал тела кнопки (без цифры, общая текстура пластика) ====== -->

File: src/entrance_group_v3/urdf/entrance_group.urdf.xacro (robot description, xacro)
@@ -1,17 +1,8 @@
 <?xml version="1.0"?>
 <!--
-  Главный xacro-файл входной группы (entrance_group_v3).
-  Система координат МОДЕЛИ:
-      +X - условно "внутрь подъезда" (домофон висит на стороне -X)
-      +Y - влево если смотреть со стороны -X (с улицы)
-      +Z - вверх
+  Главный xacro-файл входной группы (entrance_group_v3)
   При спавне в Gazebo рекомендуется задавать yaw=pi (180°), тогда
   ось -X модели совпадёт с +X мира, и наблюдатель Gazebo (стандартная
   камера со стороны +X мира) окажется СНАРУЖИ подъезда. См. launch-файл.
-  Дверь:
-      - открывается ВНУТРЬ подъезда (т.е. в направлении +X в системе модели);
-      - петли СЛЕВА (Y = +0.45 в системе модели);
-      - наружная грань двери лежит в одной плоскости с НАРУЖНОЙ стороной стены
-        (X = -0.1), т.е. дверь "вровень со стеной, на которой домофон".
 -->
 <robot xmlns:xacro="http://www.ros.org/wiki/xacro" name="entrance_group_v3">
@@ -108,5 +99,4 @@
   <!-- =====================================================
        Дверь
-       Петли СЛЕВА (Y = +0.45). Открывается ВНУТРЬ подъезда (+X).
        ===================================================== -->
   <link name="door">
@@ -131,9 +121,5 @@
     <parent link="floor"/>
     <child link="door"/>
-    <!-- Точка шарнира (петля): X=0 (в плоскости стены, нейтрально), Y=+0.45 (слева), Z=1.05. -->
     <origin xyz="${-door_x_center + door_th / 2} 0.45 1.05" rpy="0 0 0"/>
-    <!-- Ось Z. Открывается ВНУТРЬ подъезда => кромка с ручкой движется в +X.
-         С петлёй слева (Y=+0.45) для движения свободной кромки (Y=-0.9) в +X
-         нужен ПОЛОЖИТЕЛЬНЫЙ угол по оси +Z. -->
     <axis xyz="0 0 1"/>
     <limit lower="0" upper="1.57" effort="100" velocity="2.0"/>
@@ -176,6 +162,5 @@
       <geometry><cylinder radius="0.0125" length="0.3"/></geometry>
       <material name="handle_steel">
-        <!-- <color rgba="0.78 0.78 0.82 1.0"/> -->
-        <color rgba="0.68 0.68 0.72 1.0"/>
+        <color rgba="0.78 0.78 0.82 1.0"/>
       </material>
     </visual>
@@ -192,7 +177,4 @@
     <parent link="door"/>
     <child link="door_handle"/>
-    <!-- Ручка на расстоянии 80 мм от правой (свободной) кромки двери (Y=-0.82).
-         X смещаем относительно центра двери на -door_th/2 - 0.0125 (наружная сторона + радиус ручки).
-         Z = 0.05 м выше центра двери. -->
     <origin xyz="${door_th / 2.0 + 0.0125} -0.82 0.05" rpy="0 0 0"/>
   </joint>
@@ -263,28 +245,5 @@
     </visual>
   </gazebo>
-  <!-- =====================================================
-       КНОПКИ ДОМОФОНА (12 шт., через xacro-макрос)
-       ====================================================
-       Координаты ЛОКАЛЬНЫЕ относительно intercom_body.
-       Ось +X intercom_body направлена ОТ стены наружу,
-       значит лицевая грань - это X = +0.025 (полу-толщина 0.05 / 2).
-       Кнопки выступают вперёд на bx/2 = 0.004 м, итого origin.x = 0.029.
-       Раскладка телефонной клавиатуры (как видит её человек,
-       СТОЯЩИЙ ПЕРЕД ДОМОФОНОМ):
-           1  2  3
-           4  5  6
-           7  8  9
-           *  0  #
-       Эмпирически проверено на скриншоте v2: для зрителя, стоящего перед
-       домофоном, ПОЛОЖИТЕЛЬНОЕ Y модели оказывается СПРАВА.
-       Поэтому "1" (левая верхняя для зрителя) должна быть в Y=-0.018,
-       "3" - в Y=+0.018. Верхний ряд: Z МАКС положительная.
-       Шаг кнопок: 18 мм по Y, 22 мм по Z.
-       КООРДИНАТЫ (X фиксирован = 0.029, локально от intercom_body):
-         ряд 1 (Z=+0.013): 1=Y(-0.018), 2=Y(0), 3=Y(+0.018)
-         ряд 2 (Z=-0.009): 4=Y(-0.018), 5=Y(0), 6=Y(+0.018)
-         ряд 3 (Z=-0.031): 7=Y(-0.018), 8=Y(0), 9=Y(+0.018)
-         ряд 4 (Z=-0.053): *=Y(-0.018), 0=Y(0), #=Y(+0.018)
-  -->
+  <!-- Кнопки домофона -->
   <!-- Ряд 1: 1 2 3 (верхний) -->
   <xacro:intercom_button button_name="1" parent="intercom_body" xyz="0.029 -0.018  0.013"/>
