Commit message: edited robot launch pose, intercom pose in model and some fixes for dynamic control

File: src/entrance_group_v3/urdf/entrance_group.urdf.xacro (robot description, xacro)
@@ -207,8 +207,8 @@
     </visual>
     <collision>
-      <geometry><box size="0.05 0.15 0.25"/></geometry>
-    </collision>
-    <inertial>
-      <mass value="1.5"/>
+      <geometry><box size="0.015 0.12 0.20"/></geometry>
+    </collision>
+    <inertial>
+      <mass value="1.0"/>
       <inertia ixx="0.01" ixy="0" ixz="0" iyy="0.008" iyz="0" izz="0.005"/>
     </inertial>
@@ -219,5 +219,5 @@
     <!-- Домофон висит на НАРУЖНОЙ стороне стены (X = -wall_thickness/2 - depth/2 = -0.125),
          справа от двери в системе модели (Y = -0.75), высота 1.5 м. -->
-    <origin xyz="0.125 -0.75 1.5" rpy="0 0 0"/>
+    <origin xyz="0.1025 -0.75 1.4" rpy="0 0 0"/>
   </joint>
   <!-- <gazebo reference="intercom_body">

File: src/z1_model/urdf/z1_arm_macro.urdf.xacro (robot description, xacro)
@@ -295,4 +295,17 @@
           <origin xyz="0 0 0" rpy="0 0 0"/> <!-- Позиции совпадают, как вы указали -->
       </joint>
+      <!-- TCP на кончике нажимного элемента -->
+      <!-- Пустой линк без массы и визуализации -->
+      <link name="finger_tcp_link"/>
+      <!-- </link> -->
+      <joint name="finger_to_finger_tcp" type="fixed">
+        <parent link="z1_Gripper_finger"/>
+        <child link="finger_tcp_link"/>
+        <!-- Сдвигаем точку ровно туда, где находится край визуального цилиндра -->
+        <!-- Цилиндр имеет длину 0.036 и сдвинут на 0.139.
+            Eго край находится на: 0.139 + (0.036/2) = 0.157 -->
+        <origin xyz="0.157 0 -0.042" rpy="0 1.5708 0"/>
+      </joint>
+      <!-- подвижная часть схвата -->
       <joint name="${prefix}jointGripper" type="revolute">
         <origin rpy="0 0 0" xyz="0.049 0.0 0"/>

File: src/z1_model/urdf/z1_standalone_preview.urdf (robot description, URDF)
Before this commit: robot z1_model, 11 links, 10 joints
Links:
- added link finger_tcp_link
Joints:
- added joint finger_to_finger_tcp: type fixed, parent z1_Gripper_finger, child finger_tcp_link, origin xyz=0.157 0 -0.042 rpy=0 1.5708 0
