Commit message: added onboard camera and first ver of new dynamic control node (has errors)

File: src/mobile_base_model/urdf/mobile_base_macro.urdf.xacro (robot description, xacro)
@@ -202,4 +202,51 @@
                        xyz="${-wheel_x} ${-wheel_y} ${-base_h / 2.0}"
                        mass="${wheel_mass}" radius="${wheel_radius}"/>
+    <!-- Добавляем камеру -->
+    <link name="${prefix}camera_link">
+      <visual>
+        <geometry><box size="0.01 0.01 0.01"/></geometry>
+      </visual>
+      <collision>
+        <geometry><box size="0.01 0.01 0.01"/></geometry>
+      </collision>
+      <inertial>
+        <mass value="0.01"/>
+        <origin xyz="0 0 0"/>
+        <inertia ixx="1e-5" ixy="0" ixz="0" iyy="1e-5" iyz="0" izz="1e-5"/>
+      </inertial>
+    </link>
+    <joint name="${prefix}camera_joint" type="fixed">
+      <parent link="${prefix}base_link"/>
+      <child link="${prefix}camera_link"/>
+      <origin xyz="${base_l / 2.0} 0.0 ${base_h / 2.0 - 0.118}" rpy="0 0 0"/>
+    </joint>
+    <link name="${prefix}camera_optical_frame"/>
+    <joint name="${prefix}camera_optical_joint" type="fixed">
+      <parent link="${prefix}camera_link"/>
+      <child link="${prefix}camera_optical_frame"/>
+      <origin xyz="0 0 0" rpy="-1.5708 0 -1.5708"/>
+    </joint>
+    <gazebo reference="${prefix}camera_link">
+      <sensor name="${prefix}front_camera" type="camera">
+        <always_on>1</always_on>
+        <update_rate>30</update_rate>
+        <visualize>true</visualize>
+        <topic>${prefix}front_camera/raw_img</topic>
+        <camera_info_topic>${prefix}camera_info</camera_info_topic>
+        <optical_frame_id>${prefix}camera_optical_frame</optical_frame_id>
+        <camera>
+          <horizontal_fov>2.094</horizontal_fov>
+          <image>
+            <width>1920</width>
+            <height>1080</height>
+            <format>R8G8B8</format>
+          </image>
+          <clip>
+            <near>0.3</near>
+            <far>20.0</far>
+          </clip>
+        </camera>
+      </sensor>
+    </gazebo>
   </xacro:macro>
   <!-- ============================================================
