Commit message: changed platform movement type, improved platform and environment models, added new dynamic control file

File: src/delivery_dog_bringup/urdf/mobile_z1.urdf.xacro (robot description, xacro)
@@ -1,15 +1,16 @@
 <?xml version="1.0"?>
 <!--
-  Composite: мобильная mecanum-платформа + манипулятор Z1.
+  Composite: мобильная платформа (кинематический режим) + Z1.
   В этой версии:
-  * базой управляет ВСТРОЕННЫЙ плагин gz_sim::MecanumDrive (cmd_vel в GZ).
-  * Z1 управляется через gz_ros2_control + effort_controller.
-  Два плагина мирно сосуществуют в одной SDF-модели.
+    * базой управляет gz_sim::VelocityControl (cmd_vel напрямую в скорость
+      base_link). Никаких MecanumDrive, никаких ros2_control для колёс.
+    * Z1 управляется через gz_ros2_control + effort_controller.
+    * Одометрия публикуется через gz_sim::OdometryPublisher.
+  Два плагина для Z1 (ros2_control) и для базы (VelocityControl + Odometry)
+  мирно сосуществуют в одной SDF-модели.
   Аргументы:
     controllers_yaml - АБСОЛЮТНЫЙ путь к yaml для gz_ros2_control (Z1).
-                       Передаётся из launch-файла; $(find ...) в SDF не работает.
     namespace        - namespace для gz_ros2_control (контроллеров Z1).
     cmd_vel_topic    - GZ-топик для команд платформе (по умолчанию cmd_vel).
-                       Через ros_gz_bridge тот же топик доступен из ROS2.
 -->
 <robot name="mobile_z1" xmlns:xacro="http://www.ros.org/wiki/xacro">
@@ -27,5 +28,5 @@
                 xyz="0 0 ${default_mount_height / 2.0}" rpy="0 0 0"
                 use_gripper="true"/>
-  <!-- 3. ros2_control блок ТОЛЬКО для Z1 (без mobile_base_ros2_control) -->
+  <!-- 3. ros2_control блок ТОЛЬКО для Z1 -->
   <xacro:z1_ros2_control prefix="" use_gripper="true" name="Z1Hardware"/>
   <!-- 4. gz_ros2_control: 7 джойнтов Z1 -->
@@ -39,6 +40,6 @@
     </plugin>
   </gazebo>
-  <!-- 5. MecanumDrive для платформы -->
-  <xacro:mecanum_drive_plugin
+  <!-- 5. VelocityControl + OdometryPublisher для платформы -->
+  <xacro:velocity_control_plugin
       prefix=""
       topic="$(arg cmd_vel_topic)"

File: src/entrance_group_v3/urdf/entrance_group.urdf.xacro (robot description, xacro)
@@ -203,5 +203,5 @@
     <visual>
       <origin xyz="0 0 0" rpy="0 0 0"/>
-      <geometry><box size="0.05 0.15 0.25"/></geometry>
+      <geometry><box size="0.015 0.12 0.20"/></geometry>
       <material name="intercom_dark"><color rgba="0.13 0.13 0.16 1.0"/></material>
     </visual>
@@ -246,20 +246,21 @@
   </gazebo>
   <!-- Кнопки домофона -->
+  <xacro:property name="button_align" value="0.01"/>
   <!-- Ряд 1: 1 2 3 (верхний) -->
-  <xacro:intercom_button button_name="1" parent="intercom_body" xyz="0.029 -0.018  0.013"/>
-  <xacro:intercom_button button_name="2" parent="intercom_body" xyz="0.029  0.000  0.013"/>
-  <xacro:intercom_button button_name="3" parent="intercom_body" xyz="0.029  0.018  0.013"/>
+  <xacro:intercom_button button_name="1"    parent="intercom_body" xyz="${button_align} -0.018  0.013"/>
+  <xacro:intercom_button button_name="2"    parent="intercom_body" xyz="${button_align}  0.000  0.013"/>
+  <xacro:intercom_button button_name="3"    parent="intercom_body" xyz="${button_align}  0.018  0.013"/>
   <!-- Ряд 2: 4 5 6 -->
-  <xacro:intercom_button button_name="4" parent="intercom_body" xyz="0.029 -0.018 -0.009"/>
-  <xacro:intercom_button button_name="5" parent="intercom_body" xyz="0.029  0.000 -0.009"/>
-  <xacro:intercom_button button_name="6" parent="intercom_body" xyz="0.029  0.018 -0.009"/>
+  <xacro:intercom_button button_name="4"    parent="intercom_body" xyz="${button_align} -0.018 -0.009"/>
+  <xacro:intercom_button button_name="5"    parent="intercom_body" xyz="${button_align}  0.000 -0.009"/>
+  <xacro:intercom_button button_name="6"    parent="intercom_body" xyz="${button_align}  0.018 -0.009"/>
   <!-- Ряд 3: 7 8 9 -->
-  <xacro:intercom_button button_name="7" parent="intercom_body" xyz="0.029 -0.018 -0.031"/>
-  <xacro:intercom_button button_name="8" parent="intercom_body" xyz="0.029  0.000 -0.031"/>
-  <xacro:intercom_button button_name="9" parent="intercom_body" xyz="0.029  0.018 -0.031"/>
+  <xacro:intercom_button button_name="7"    parent="intercom_body" xyz="${button_align} -0.018 -0.031"/>
+  <xacro:intercom_button button_name="8"    parent="intercom_body" xyz="${button_align}  0.000 -0.031"/>
+  <xacro:intercom_button button_name="9"    parent="intercom_body" xyz="${button_align}  0.018 -0.031"/>
   <!-- Ряд 4: * 0 # (нижний) -->
-  <xacro:intercom_button button_name="star" parent="intercom_body" xyz="0.029 -0.018 -0.053"/>
-  <xacro:intercom_button button_name="0"    parent="intercom_body" xyz="0.029  0.000 -0.053"/>
-  <xacro:intercom_button button_name="hash" parent="intercom_body" xyz="0.029  0.018 -0.053"/>
+  <xacro:intercom_button button_name="star" parent="intercom_body" xyz="${button_align} -0.018 -0.053"/>
+  <xacro:intercom_button button_name="0"    parent="intercom_body" xyz="${button_align}  0.000 -0.053"/>
+  <xacro:intercom_button button_name="hash" parent="intercom_body" xyz="${button_align}  0.018 -0.053"/>
   <!-- <xacro:include filename="buts.xacro"/> -->
 </robot>

File: src/mobile_base_model/urdf/mobile_base_macro.urdf.xacro (robot description, xacro)
@@ -1,49 +1,43 @@
 <?xml version="1.0"?>
 <!--
-  Mobile base macro (mecanum, 4 колеса).
-  ИЗМЕНЕНО относительно предыдущей версии: добавлен макрос xacro:mecanum_drive_plugin,
-  который вставляет встроенный плагин gz_sim::systems::MecanumDrive.
-  Он работает на УРОВНЕ Gazebo: получает /cmd_vel, сам считает кинематику
-  и прикладывает силы к корпусу - в результате платформа реально едет вбок
-  (без моделирования роликов на колёсах).
-  Параметры макроса xacro:mobile_base те же.
-  Новый макрос: xacro:mecanum_drive_plugin
-    prefix       - префикс колёсных джойнтов (например "" или "mb_")
-    topic        - топик cmd_vel (по умолчанию /cmd_vel)
-    odom_topic   - публикация odom (по умолчанию /odom)
-    wheel_separation - расстояние между левой и правой парой (м)
-    wheelbase        - расстояние между передней и задней парой (м)
-    wheel_radius     - радиус колеса (м)
+  Mobile base macro (kinematic режим VelocityControl + OdometryPublisher).
+  =========================================================================
+  В этой версии:
+    * НЕТ MecanumDrive, НЕТ ros2_control блока для колёс.
+    * gz_sim::systems::VelocityControl слушает /cmd_vel (GZ-топик) и НАПРЯМУЮ
+      задаёт линейную и угловую скорость base_link. Это кинематический режим:
+      робот идеально следует cmd_vel, без проскальзываний.
+    * gz_sim::systems::OdometryPublisher публикует /odom (GZ-топик) по реальной
+      позе base_link относительно odom-фрейма + TF одометрии.
+    * 4 колеса оставлены ВИЗУАЛЬНО как раньше, но их collision отключён
+      и они подвешены через fixed-джойнты - не влияют на физику.
+    * 3 кастера-шарика с почти нулевым трением держат корпус над полом
+      (без них VelocityControl может конфликтовать с гравитацией на старте).
+  Макрос xacro:mobile_base принимает те же параметры, что и раньше.
+  Старый макрос mecanum_drive_plugin удалён, добавлен velocity_control_plugin.
 -->
 <robot xmlns:xacro="http://www.ros.org/wiki/xacro">
-  <!-- ====== Параметры по умолчанию (можно переопределять при вызове макроса) ====== -->
-  <!-- <xacro:property name="default_base_l"        value="0.60"/>
-  <xacro:property name="default_base_w"        value="0.40"/>
-  <xacro:property name="default_base_h"        value="0.20"/> -->
+  <!-- ====== Параметры по умолчанию ====== -->
   <xacro:property name="default_base_l"        value="1.00"/>
   <xacro:property name="default_base_w"        value="0.45"/>
   <xacro:property name="default_base_h"        value="0.545"/>
   <xacro:property name="default_base_mass"     value="30.0"/>
-  <!-- <xacro:property name="default_wheel_radius"  value="0.080"/> -->
   <xacro:property name="default_wheel_radius"  value="0.10"/>
   <xacro:property name="default_wheel_thick"   value="0.050"/>
   <xacro:property name="default_wheel_mass"    value="1.0"/>
-  <!-- <xacro:property name="default_wheel_x"       value="0.22"/>
-  <xacro:property name="default_wheel_y"       value="0.20"/> -->
   <xacro:property name="default_wheel_x"       value="${default_base_l / 2.0 - default_wheel_radius}"/>
   <xacro:property name="default_wheel_y"       value="${default_base_w / 2.0}"/>
-  <!-- <xacro:property name="default_mount_height"  value="0.02"/> -->
   <xacro:property name="default_mount_height"  value="0.14"/>
-  <!-- ==== my ==== -->
   <xacro:property name="default_mount_lingth"  value="0.2"/>
-  <xacro:property name="default_mount_x"  value="${(default_base_l - default_mount_lingth) / 2.0}"/>
-  <!-- ====== Локальный макрос: одно колесо ====== -->
-  <xacro:macro name="mecanum_wheel"
-               params="prefix name xyz mass radius thick">
-    <link name="${prefix}wheel_${name}_link">
-      <visual>
-        <origin xyz="0 0 0" rpy="${pi/2} 0 0"/>
-        <geometry>
-          <cylinder radius="${radius}" length="${thick}"/>
+  <xacro:property name="default_mount_x"       value="${(default_base_l - default_mount_lingth) / 2.0}"/>
+  <!-- ====== Локальный макрос: кастер-шарик с нулевым трением ====== -->
+  <xacro:macro name="caster_ball" params="prefix name xyz mass radius">
+    <xacro:property name="ball_inertia" value="${ (2/5) * mass * radius * radius }"/>
+    <link name="${prefix}caster_${name}">
+      <visual>
+        <origin xyz="0 0 0" rpy="0 0 0"/>
+        <geometry>
+          <sphere radius="${radius}"/>
+          <!-- <cylinder radius="${radius}"/> -->
         </geometry>
         <material name="${prefix}wheel_mat">
@@ -52,30 +46,32 @@
       </visual>
       <collision>
-        <origin xyz="0 0 0" rpy="${pi/2} 0 0"/>
-        <geometry>
-          <cylinder radius="${radius}" length="${thick}"/>
-        </geometry>
+        <geometry>
+          <sphere radius="${radius}"/>
+        </geometry>
+        <surface>
+          <friction>
+            <ode>
+              <mu>0.00001</mu>
+              <mu2>0.00001</mu2>
+            </ode>
+          </friction>
+        </surface>
       </collision>
+      <!-- <visual>
+        <geometry>
+          <sphere radius="0.005"/>
+        </geometry>
+      </visual> -->
       <inertial>
         <mass value="${mass}"/>
-        <inertia
-          ixx="${mass*(3*radius*radius + thick*thick)/12.0}"
-          iyy="${mass*radius*radius/2.0}"
-          izz="${mass*(3*radius*radius + thick*thick)/12.0}"
-          ixy="0" ixz="0" iyz="0"/>
+        <inertia ixx="${ball_inertia}" iyy="${ball_inertia}" izz="${ball_inertia}" ixy="0" ixz="0" iyz="0"/>
       </inertial>
     </link>
-    <joint name="${prefix}wheel_${name}_joint" type="continuous">
+    <joint name="${prefix}caster_${name}_joint" type="fixed">
       <parent link="${prefix}base_link"/>
-      <child  link="${prefix}wheel_${name}_link"/>
-      <origin xyz="${xyz}" rpy="0 0 0"/>
-      <axis xyz="0 1 0"/>
-      <dynamics damping="0.05" friction="0.1"/>
+      <child  link="${prefix}caster_${name}"/>
+      <origin xyz="${xyz}"/>
     </joint>
-    <gazebo reference="${prefix}wheel_${name}_link">
-      <mu1>1.0</mu1>
-      <mu2>1.0</mu2>
-      <kp>1e7</kp>
-      <kd>10.0</kd>
+    <gazebo reference="${prefix}caster_${name}">
       <visual>
         <material>
@@ -84,4 +80,6 @@
         </material>
       </visual>
+      <mu1>0.00001</mu1>
+      <mu2>0.00001</mu2>
     </gazebo>
   </xacro:macro>
@@ -134,6 +132,8 @@
     </link>
     <gazebo reference="${prefix}base_link">
-      <mu1>0.3</mu1>
-      <mu2>0.3</mu2>
+      <!-- Низкое трение корпуса по самому себе - на случай, если уголок
+           коснётся земли при наклоне. -->
+      <mu1>0.1</mu1>
+      <mu2>0.1</mu2>
       <visual>
         <material>
@@ -168,44 +168,50 @@
       <parent link="${prefix}base_link"/>
       <child  link="${prefix}z1_mount"/>
-      <!-- Сидит на крышке корпуса по центру. -->
       <origin xyz="${default_mount_x} 0 ${base_h/2.0 + mount_height/2.0}" rpy="0 0 0"/>
     </joint>
-    <!-- ================== 4 колеса ================== -->
-    <!-- Локальные координаты колёс относительно base_link.
-         Z колеса = -base_h/2 (низ корпуса) - НЕТ, центр колеса на той же высоте,
-         что и нижняя грань корпуса. Низ колеса (z = z_wheel - radius) лежит на земле. -->
+    <!-- ================== 4 ВИЗУАЛЬНЫХ колеса ================== -->
     <xacro:property name="wheel_z_local" value="${-base_h/2.0}"/>
-    <xacro:mecanum_wheel prefix="${prefix}" name="fl"
-                         xyz="${ wheel_x}  ${ wheel_y} ${wheel_z_local}"
-                         mass="${wheel_mass}" radius="${wheel_radius}" thick="${wheel_thick}"/>
-    <xacro:mecanum_wheel prefix="${prefix}" name="fr"
-                         xyz="${ wheel_x} ${-wheel_y} ${wheel_z_local}"
-                         mass="${wheel_mass}" radius="${wheel_radius}" thick="${wheel_thick}"/>
-    <xacro:mecanum_wheel prefix="${prefix}" name="rl"
-                         xyz="${-wheel_x}  ${ wheel_y} ${wheel_z_local}"
-                         mass="${wheel_mass}" radius="${wheel_radius}" thick="${wheel_thick}"/>
-    <xacro:mecanum_wheel prefix="${prefix}" name="rr"
-                         xyz="${-wheel_x} ${-wheel_y} ${wheel_z_local}"
-                         mass="${wheel_mass}" radius="${wheel_radius}" thick="${wheel_thick}"/>
+    <!-- <xacro:dummy_wheel prefix="${prefix}" name="fl"
+                       xyz="${ wheel_x}  ${ wheel_y} ${wheel_z_local}"
+                       mass="${wheel_mass}" radius="${wheel_radius}" thick="${wheel_thick}"/>
+    <xacro:dummy_wheel prefix="${prefix}" name="fr"
+                       xyz="${ wheel_x} ${-wheel_y} ${wheel_z_local}"
+                       mass="${wheel_mass}" radius="${wheel_radius}" thick="${wheel_thick}"/>
+    <xacro:dummy_wheel prefix="${prefix}" name="rl"
+                       xyz="${-wheel_x}  ${ wheel_y} ${wheel_z_local}"
+                       mass="${wheel_mass}" radius="${wheel_radius}" thick="${wheel_thick}"/>
+    <xacro:dummy_wheel prefix="${prefix}" name="rr"
+                       xyz="${-wheel_x} ${-wheel_y} ${wheel_z_local}"
+                       mass="${wheel_mass}" radius="${wheel_radius}" thick="${wheel_thick}"/> -->
+    <!-- ================== 3 кастера-шарика ================== -->
+    <!-- Низ корпуса лежит на z = -base_h/2. Кастеры висят чуть ниже,
+         чтобы они касались земли, а корпус - нет.
+         z_caster_local = -base_h/2 - wheel_radius + 0.005
+         (сфера радиуса 0.005 должна касаться z=0 при footprint=z=0). -->
+    <!-- <xacro:property name="caster_z" value="${-base_h/2.0 - wheel_radius + 0.005}"/> -->
+    <xacro:caster_ball prefix="${prefix}" name="fl"
+                       xyz="${ wheel_x}  ${ wheel_y} ${-base_h / 2.0}"
+                       mass="${wheel_mass}" radius="${wheel_radius}"/>
+    <xacro:caster_ball prefix="${prefix}" name="fr"
+                       xyz="${ wheel_x} ${-wheel_y} ${-base_h / 2.0}"
+                       mass="${wheel_mass}" radius="${wheel_radius}"/>
+    <xacro:caster_ball prefix="${prefix}" name="rl"
+                       xyz="${-wheel_x}  ${ wheel_y} ${-base_h / 2.0}"
+                       mass="${wheel_mass}" radius="${wheel_radius}"/>
+    <xacro:caster_ball prefix="${prefix}" name="rr"
+                       xyz="${-wheel_x} ${-wheel_y} ${-base_h / 2.0}"
+                       mass="${wheel_mass}" radius="${wheel_radius}"/>
   </xacro:macro>
   <!-- ============================================================
-       ВСТРОЕННЫЙ ПЛАГИН gz_sim MecanumDrive.
-       Принимает /cmd_vel прямо в Gazebo, без ros_gz_bridge не нужен
-       Twist-to-wheels: плагин сам прикладывает корректные усилия
-       к корпусу, обеспечивая mecanum-движение в любую сторону.
+       ВСТРОЕННЫЕ ПЛАГИНЫ: VelocityControl + OdometryPublisher.
        Параметры:
-         prefix             - префикс джойнтов колёс
-         topic              - имя топика cmd_vel (по умолчанию /cmd_vel,
-                              ВНИМАНИЕ: это GZ-топик, для управления из ROS2
-                              его нужно прокинуть через ros_gz_bridge)
-         odom_topic         - публикация odom (GZ-топик)
-         tf_topic           - публикация TF (GZ-топик)
-         frame_id           - имя odom-фрейма
-         child_frame_id     - имя base-фрейма для одометрии
-         wheel_separation_x - расстояние между передней и задней парой (м)
-         wheel_separation_y - расстояние между левой и правой парой (м)
-         wheel_radius       - радиус колеса (м)
+         topic              - GZ-топик для cmd_vel (default: cmd_vel).
+                              Через ros_gz_bridge доступен из ROS2.
+         odom_topic         - GZ-топик одометрии (default: odom).
+         tf_topic           - GZ-топик TF (default: tf).
+         frame_id           - имя odom-фрейма.
+         child_frame_id     - имя base-фрейма для одометрии.
        ============================================================ -->
-  <xacro:macro name="mecanum_drive_plugin"
+  <xacro:macro name="velocity_control_plugin"
                params="prefix:=''
                        topic:='cmd_vel'
@@ -214,55 +220,22 @@
                        frame_id:='odom'
                        child_frame_id:='base_footprint'
-                       wheel_separation_x:=${2.0*default_wheel_x}
-                       wheel_separation_y:=${2.0*default_wheel_y}
-                       wheel_radius:=${default_wheel_radius}">
+                       odom_pub_frequency:='50'">
     <gazebo>
-      <plugin filename="gz-sim-mecanum-drive-system"
-              name="gz::sim::systems::MecanumDrive">
-        <front_left_joint>${prefix}wheel_fl_joint</front_left_joint>
-        <front_right_joint>${prefix}wheel_fr_joint</front_right_joint>
-        <back_left_joint>${prefix}wheel_rl_joint</back_left_joint>
-        <back_right_joint>${prefix}wheel_rr_joint</back_right_joint>
-        <wheel_separation>${wheel_separation_y}</wheel_separation>
-        <wheelbase>${wheel_separation_x}</wheelbase>
-        <wheel_radius>${wheel_radius}</wheel_radius>
+      <!-- 1. VelocityControl: cmd_vel напрямую в скорость base_link -->
+      <plugin filename="gz-sim-velocity-control-system"
+              name="gz::sim::systems::VelocityControl">
         <topic>${topic}</topic>
+      </plugin>
+      <!-- 2. OdometryPublisher: реальная поза base_link -> /odom + TF -->
+      <plugin filename="gz-sim-odometry-publisher-system"
+              name="gz::sim::systems::OdometryPublisher">
+        <odom_frame>${frame_id}</odom_frame>
+        <robot_base_frame>${prefix}base_link</robot_base_frame>
+        <odom_publish_frequency>${odom_pub_frequency}</odom_publish_frequency>
         <odom_topic>${odom_topic}</odom_topic>
         <tf_topic>${tf_topic}</tf_topic>
-        <frame_id>${frame_id}</frame_id>
-        <child_frame_id>${child_frame_id}</child_frame_id>
-        <odom_publish_frequency>50</odom_publish_frequency>
+        <dimensions>3</dimensions>
       </plugin>
     </gazebo>
   </xacro:macro>
-  <!-- ============================================================
-       Старый ros2_control блок для платформы оставлен, на случай
-       если когда-нибудь захочется управлять колёсами явно. Сейчас
-       НЕ используется (см. mobile_base_standalone.urdf.xacro и
-       mobile_z1.urdf.xacro - там подключается mecanum_drive_plugin
-       вместо ros2_control).
-       ============================================================ -->
-  <xacro:macro name="mobile_base_ros2_control"
-               params="prefix:='' name:=MobileBaseGazeboSystem">
-    <ros2_control name="${name}" type="system">
-      <hardware>
-        <plugin>gz_ros2_control/GazeboSimSystem</plugin>
-      </hardware>
-      <xacro:wheel_iface name="${prefix}wheel_fl_joint"/>
-      <xacro:wheel_iface name="${prefix}wheel_fr_joint"/>
-      <xacro:wheel_iface name="${prefix}wheel_rl_joint"/>
-      <xacro:wheel_iface name="${prefix}wheel_rr_joint"/>
-    </ros2_control>
-  </xacro:macro>
-  <xacro:macro name="wheel_iface" params="name">
-    <joint name="${name}">
-      <command_interface name="velocity">
-        <param name="min">-30.0</param>
-        <param name="max"> 30.0</param>
-      </command_interface>
-      <state_interface name="position"/>
-      <state_interface name="velocity"/>
-      <state_interface name="effort"/>
-    </joint>
-  </xacro:macro>
 </robot>

File: src/mobile_base_model/urdf/mobile_base_standalone.urdf.xacro (robot description, xacro)
@@ -2,6 +2,6 @@
 <!--
   Standalone-сборка одной только мобильной платформы (без Z1).
-  Использует встроенный плагин gz_sim::MecanumDrive (а не ros2_control)
-  для управления через /cmd_vel.
+  Использует gz_sim::VelocityControl + gz_sim::OdometryPublisher
+  для управления через /cmd_vel и публикации одометрии.
   ВНИМАНИЕ: топик cmd_vel здесь - это GZ-топик. Чтобы публиковать в него
   из ROS2, нужен ros_gz_bridge (он же поднимается в launch).
@@ -10,7 +10,6 @@
   <xacro:include filename="mobile_base_macro.urdf.xacro"/>
   <xacro:mobile_base prefix=""/>
-  <!-- Кинематика mecanum через встроенный плагин Gazebo.
-       Топик GZ /cmd_vel пробрасывается в ROS2 через ros_gz_bridge в launch. -->
-  <xacro:mecanum_drive_plugin
+  <!-- Кинематический drive через встроенные плагины Gazebo. -->
+  <xacro:velocity_control_plugin
       prefix=""
       topic="cmd_vel"
