Commit message: added 'finger' to gripper, fixed dynamic control node, added flag to turn on sim cameras

File: src/delivery_dog_bringup/urdf/mobile_z1.urdf.xacro (robot description, xacro)
@@ -16,10 +16,11 @@
 <robot name="mobile_z1" xmlns:xacro="http://www.ros.org/wiki/xacro">
   <xacro:property name="default_mount_height"  value="0.14"/>
-  <xacro:arg name="controllers_yaml" default="/tmp/mobile_z1_controllers.yaml"/>
-  <xacro:arg name="namespace"        default="/robot"/>
-  <xacro:arg name="cmd_vel_topic"    default="cmd_vel"/>
+  <xacro:arg name="controllers_yaml"  default="/tmp/mobile_z1_controllers.yaml"/>
+  <xacro:arg name="namespace"         default="/robot"/>
+  <xacro:arg name="cmd_vel_topic"     default="cmd_vel"/>
+  <xacro:arg name="cameras_on"        default="false"/>
   <!-- 1. Платформа -->
   <xacro:include filename="$(find mobile_base_model)/urdf/mobile_base_macro.urdf.xacro"/>
-  <xacro:mobile_base prefix="" mount_height="${default_mount_height}"/>
+  <xacro:mobile_base prefix="" mount_height="${default_mount_height}" cameras_on="$(arg cameras_on)"/>
   <!-- 2. Z1 на крышке -->
   <xacro:include filename="$(find z1_model)/urdf/z1_arm_macro.urdf.xacro"/>

File: src/mobile_base_model/urdf/mobile_base_macro.urdf.xacro (robot description, xacro)
@@ -31,4 +31,6 @@
   <xacro:property name="default_mount_lingth"  value="0.2"/>
   <xacro:property name="default_mount_x"       value="${(default_base_l - default_mount_lingth) / 2.0}"/>
+  <xacro:property name="lidar_offset_x"       value="0.013"/>
+  <xacro:property name="default_cameras_on"   value="false"/>
   <!-- ====== Локальный макрос: кастер-шарик с нулевым трением ====== -->
   <xacro:macro name="caster_ball" params="prefix name xyz mass radius">
@@ -96,5 +98,7 @@
                        wheel_x:=${default_wheel_x}
                        wheel_y:=${default_wheel_y}
-                       mount_height:=${default_mount_height}">
+                       mount_height:=${default_mount_height}
+                       mount_height:=${default_mount_height}
+                       cameras_on:=${default_cameras_on}">
     <!-- ================== base_footprint (на полу) ================== -->
     <link name="${prefix}base_footprint"/>
@@ -168,5 +172,5 @@
       <parent link="${prefix}base_link"/>
       <child  link="${prefix}z1_mount"/>
-      <origin xyz="${default_mount_x} 0 ${base_h/2.0 + mount_height/2.0}" rpy="0 0 0"/>
+      <origin xyz="${default_mount_x - lidar_offset_x} 0 ${base_h/2.0 + mount_height/2.0}" rpy="0 0 0"/>
     </joint>
     <!-- ================== 4 ВИЗУАЛЬНЫХ колеса ================== -->
@@ -203,50 +207,56 @@
                        mass="${wheel_mass}" radius="${wheel_radius}"/>
     <!-- Добавляем камеру -->
-    <link name="${prefix}camera_link">
-      <visual>
-        <geometry><box size="0.01 0.01 0.01"/></geometry>
-      </visual>
-      <collision>
-        <geometry><box size="0.01 0.01 0.01"/></geometry>
-      </collision>
-      <inertial>
-        <mass value="0.01"/>
-        <origin xyz="0 0 0"/>
-        <inertia ixx="1e-5" ixy="0" ixz="0" iyy="1e-5" iyz="0" izz="1e-5"/>
-      </inertial>
-    </link>
-    <joint name="${prefix}camera_joint" type="fixed">
-      <parent link="${prefix}base_link"/>
-      <child link="${prefix}camera_link"/>
-      <origin xyz="${base_l / 2.0} 0.0 ${base_h / 2.0 - 0.118}" rpy="0 0 0"/>
-    </joint>
-    <link name="${prefix}camera_optical_frame"/>
-    <joint name="${prefix}camera_optical_joint" type="fixed">
-      <parent link="${prefix}camera_link"/>
-      <child link="${prefix}camera_optical_frame"/>
-      <origin xyz="0 0 0" rpy="-1.5708 0 -1.5708"/>
-    </joint>
-    <gazebo reference="${prefix}camera_link">
-      <sensor name="${prefix}front_camera" type="camera">
-        <always_on>1</always_on>
-        <update_rate>30</update_rate>
-        <visualize>true</visualize>
-        <topic>${prefix}front_camera/raw_img</topic>
-        <camera_info_topic>${prefix}camera_info</camera_info_topic>
-        <optical_frame_id>${prefix}camera_optical_frame</optical_frame_id>
-        <camera>
-          <horizontal_fov>2.094</horizontal_fov>
-          <image>
-            <width>1920</width>
-            <height>1080</height>
-            <format>R8G8B8</format>
-          </image>
-          <clip>
-            <near>0.3</near>
-            <far>20.0</far>
-          </clip>
-        </camera>
-      </sensor>
-    </gazebo>
+    <xacro:if value="${cameras_on == 'true'}">
+      <link name="${prefix}my_camera_link">
+        <visual>
+          <geometry><box size="0.01 0.01 0.01"/></geometry>
+        </visual>
+        <collision>
+          <geometry><box size="0.01 0.01 0.01"/></geometry>
+        </collision>
+        <inertial>
+          <mass value="0.01"/>
+          <origin xyz="0 0 0"/>
+          <inertia ixx="1e-5" ixy="0" ixz="0" iyy="1e-5" iyz="0" izz="1e-5"/>
+        </inertial>
+      </link>
+      <joint name="${prefix}my_camera_joint" type="fixed">
+        <parent link="${prefix}base_link"/>
+        <child link="${prefix}my_camera_link"/>
+        <!-- <origin xyz="${base_l / 2.0} 0.0 ${base_h / 2.0 - 0.118}" rpy="0 0 0"/> -->
+        <origin xyz="${base_l / 2.0 - lidar_offset_x} 0.0 ${base_h / 2.0 + default_mount_height}" rpy="0 -0.837468 0"/>
+      </joint>
+      <link name="${prefix}my_camera_optical_frame"/>
+      <joint name="${prefix}my_camera_optical_joint" type="fixed">
+        <parent link="${prefix}my_camera_link"/>
+        <child link="${prefix}my_camera_optical_frame"/>
+        <origin xyz="0 0 0" rpy="-1.5708 0 -1.5708"/>
+      </joint>
+      <gazebo reference="${prefix}my_camera_link">
+        <sensor name="${prefix}sensor_my_camera" type="camera">
+          <always_on>1</always_on>
+          <update_rate>30</update_rate>
+          <visualize>true</visualize>
+          <topic>${prefix}sensor_my_camera/raw_img</topic>
+          <camera_info_topic>${prefix}my_camera_info</camera_info_topic>
+          <optical_frame_id>${prefix}my_camera_optical_frame</optical_frame_id>
+          <camera>
+            <!-- <horizontal_fov>2.094</horizontal_fov> -->
+            <vertical_fov>0.733038</vertical_fov>
+            <image>
+              <!-- <width>1920</width>
+              <height>1080</height> -->
+              <width>2160</width>
+              <height>3840</height>
+              <format>R8G8B8</format>
+            </image>
+            <clip>
+              <near>0.3</near>
+              <far>20.0</far>
+            </clip>
+          </camera>
+        </sensor>
+      </gazebo>
+    </xacro:if>
   </xacro:macro>
   <!-- ============================================================

File: src/z1_model/urdf/z1_arm_macro.urdf.xacro (robot description, xacro)
@@ -260,4 +260,39 @@
         </inertial>
       </link>
+      <!-- Нажимной элемент (Finger) -->
+      <link name="z1_Gripper_finger">
+        <inertial>
+            <origin xyz="0.117494 0.0 -0.040887" rpy="0 0 0"/>
+            <mass value="0.003286"/>
+            <inertia
+                ixx="0.0000000259" ixy="0.0" ixz="-0.0000000568"
+                iyy="0.000001303" iyz="0.0"
+                izz="0.000001293"/>
+        </inertial>
+        <visual>
+            <!-- <origin xyz="0 0 0" rpy="0 0 0"/> -->
+            <origin xyz="0.139 0 -0.042" rpy="0 1.5708 0"/>
+            <geometry>
+                <!-- <mesh filename="$(find z1_model)/meshes/visual/stl_models/z1_Gripper_finger.stl" scale="1 1 1"/> -->
+                <cylinder length="0.036" radius="0.003"/>
+            </geometry>
+            <material name="grey"/>
+        </visual>
+        <collision>
+            <!-- <origin xyz="0 0 0" rpy="0 0 0"/> -->
+            <origin xyz="0.139 0 -0.042" rpy="0 1.5708 0"/>
+            <geometry>
+                <!-- Рекомендуется использовать упрощенную геометрию для коллизий, но можно и stl -->
+                <!-- <mesh filename="$(find z1_model)/meshes/visual/z1_Gripper_finger.stl" scale="1 1 1"/> -->
+                <cylinder length="0.036" radius="0.003"/>
+            </geometry>
+        </collision>
+      </link>
+      <!-- Крепление нажимного элемента к статору схвата -->
+      <joint name="gripper_stator_to_finger" type="fixed">
+          <parent link="gripperStator"/> <!-- Замените на точное имя link'а вашего статора -->
+          <child link="z1_Gripper_finger"/>
+          <origin xyz="0 0 0" rpy="0 0 0"/> <!-- Позиции совпадают, как вы указали -->
+      </joint>
       <joint name="${prefix}jointGripper" type="revolute">
         <origin rpy="0 0 0" xyz="0.049 0.0 0"/>

File: src/z1_model/urdf/z1_model.urdf.xacro (robot description, xacro)
@@ -254,4 +254,39 @@
             </inertial>
         </link>
+        <!-- Нажимной элемент (Finger) -->
+      <link name="z1_Gripper_finger">
+        <inertial>
+            <origin xyz="0.117494 0.0 -0.040887" rpy="0 0 0"/>
+            <mass value="0.003286"/>
+            <inertia
+                ixx="0.0000000259" ixy="0.0" ixz="-0.0000000568"
+                iyy="0.000001303" iyz="0.0"
+                izz="0.000001293"/>
+        </inertial>
+        <visual>
+            <!-- <origin xyz="0 0 0" rpy="0 0 0"/> -->
+            <origin xyz="0.139 0 -0.042" rpy="0 1.5708 0"/>
+            <geometry>
+                <!-- <mesh filename="$(find z1_model)/meshes/visual/stl_models/z1_Gripper_finger.stl" scale="1 1 1"/> -->
+                <cylinder length="0.036" radius="0.003"/>
+            </geometry>
+            <material name="grey"/>
+        </visual>
+        <collision>
+            <!-- <origin xyz="0 0 0" rpy="0 0 0"/> -->
+            <origin xyz="0.139 0 -0.042" rpy="0 1.5708 0"/>
+            <geometry>
+                <!-- Рекомендуется использовать упрощенную геометрию для коллизий, но можно и stl -->
+                <!-- <mesh filename="$(find z1_model)/meshes/visual/z1_Gripper_finger.stl" scale="1 1 1"/> -->
+                <cylinder length="0.036" radius="0.003"/>
+            </geometry>
+        </collision>
+      </link>
+      <!-- Крепление нажимного элемента к статору схвата -->
+      <joint name="gripper_stator_to_finger" type="fixed">
+          <parent link="gripperStator"/> <!-- Замените на точное имя link'а вашего статора -->
+          <child link="z1_Gripper_finger"/>
+          <origin xyz="0 0 0" rpy="0 0 0"/> <!-- Позиции совпадают, как вы указали -->
+      </joint>
         <joint name="jointGripper" type="revolute">
             <origin rpy="0 0 0" xyz="0.049 0.0 0"/>
