Commit message: added bracet and d_box in full model, added mujoco folder with entrance model

File: src/delivery_dog_bringup/urdf/b2_z1.urdf.xacro (robot description, xacro)
@@ -10,16 +10,71 @@
     <!-- <xacro:arg name="b2_xyz" default="0 0 0"/>
     <xacro:arg name="b2_rpy" default="0 0 0"/> -->
-    <xacro:arg name="mount_position" default="0.35 0 0.275"/> <!-- высота крепления Z1 над спиной -->
+    <xacro:arg name="mount_position" default="0.1945 0 0.276"/> <!-- 0.361 высота крепления Z1 над спиной -->
     <!-- Вставляем собаку B2 (без ros2_control) -->
     <xacro:b2_robot prefix="b2_"/>
     <!-- xyz="$(arg b2_xyz)" rpy="$(arg b2_rpy)" -->
+    <link name="bracket">
+        <visual>
+            <origin rpy="0 0 0" xyz="0 0 0"/>
+            <geometry>
+                <mesh filename="$(find delivery_dog_bringup)/meshes/bracket2.stl" scale="0.001 0.001 0.001"/>
+            </geometry>
+            <material name="iron_gold"/>
+        </visual>
+        <collision>
+            <geometry>
+                <box size="0.128 0.16 0.185"/>
+            </geometry>
+            <origin rpy="0 0 0" xyz="-0.1945 0 0.1805"/>
+        </collision>
+        <inertial>
+            <origin xyz="0.194501 0.0 0.174264" rpy="0 0 0"/>
+            <mass value="3.603948"/>
+            <inertia ixx="0.031873" ixy="0.0" ixz="0.0" iyy="0.022245" iyz="0.0" izz="0.019470"/>
+        </inertial>
+    </link>
+    <joint name="bracket_joint" type="fixed">
+        <origin xyz="0 0 0" rpy="0 0 0"/>
+        <parent link="b2_trunk"/>
+        <child link="bracket"/>
+    </joint>
+    <link name="delivery_box">
+        <visual>
+            <origin rpy="0 0 0" xyz="0 0 0"/>
+            <geometry>
+                <box size="0.395 0.32 0.26"/>
+            </geometry>
+            <material name="grey"/>
+        </visual>
+        <collision>
+            <origin rpy="0 0 0" xyz="0 0 0"/>
+            <geometry>
+                <box size="0.395 0.32 0.26"/>
+            </geometry>
+        </collision>
+        <inertial>
+            <origin rpy="0 0 0" xyz="0 0 0"/>
+            <mass value="15.0"/>
+            <inertia ixx="0.1845" ixy="0.0" ixz="0.0" iyy="0.247781" iyz="0.0" izz="0.288281"/>
+        </inertial>
+    </link>
+    <joint name="delivery_box_joint" type="fixed">
+        <origin rpy="0 0 0" xyz="-0.28 0 0.22"/>
+        <parent link="b2_trunk"/>
+        <child link="delivery_box"/>
+    </joint>
     <!-- Создаём отдельный линк для крепления Z1 -->
     <link name="z1_mount"/>
     <!-- Крепим монтажную площадку к trunk собаки (подбираем координаты) -->
     <joint name="z1_mount_joint" type="fixed">
-    <origin xyz="$(arg mount_position)" rpy="0 0 0"/>
-    <parent link="b2_trunk"/>
-    <child link="z1_mount"/>
+        <origin xyz="$(arg mount_position)" rpy="0 0 0"/>
+        <parent link="b2_trunk"/>
+        <child link="z1_mount"/>
     </joint>
+    <!-- <joint name="z1_mount_joint" type="fixed">
+        <origin xyz="0 0 0.0925" rpy="0 0 0"/>
+        <parent link="bracket"/>
+        <child link="z1_mount"/>
+    </joint> -->
     <!-- Устанавливаем манипулятор Z1 на монтажную площадку -->
     <xacro:z1_arm prefix="z1_"

File: src/delivery_dog_bringup/urdf/b2_z1_rel_preview.urdf (robot description, URDF)
Before this commit: robot b2_z1, 46 links, 45 joints
Links:
- added link bracket, mass 3.603948; collision box size=0.128 0.16 0.185; visual mesh filename=../meshes/bracket2.stl scale=0.001 0.001 0.001
- added link delivery_box, mass 15.0; collision box size=0.395 0.32 0.26; visual box size=0.395 0.32 0.26
Joints:
- added joint bracket_joint: type fixed, parent b2_trunk, child bracket, origin xyz=0 0 0 rpy=0 0 0
- added joint delivery_box_joint: type fixed, parent b2_trunk, child delivery_box, origin xyz=-0.28 0 0.22 rpy=0 0 0
- joint z1_mount_joint: origin xyz=0.35 0 0.275 rpy=0 0 0 -> xyz=0.1945 0 0.276 rpy=0 0 0

Commit message: fixed bracket collision and temp changes for dog mujoco xml

File: src/delivery_dog_bringup/urdf/b2_z1.urdf.xacro (robot description, xacro)
@@ -26,5 +26,5 @@
                 <box size="0.128 0.16 0.185"/>
             </geometry>
-            <origin rpy="0 0 0" xyz="-0.1945 0 0.1805"/>
+            <origin rpy="0 0 0" xyz="0.1945 0 0.1805"/>
         </collision>
         <inertial>
