Commit message: added B2 macros and standalone urdf, deleted test files

File: src/b2_description/xacro/leg.xacro (robot description, xacro)
@@ -2,5 +2,5 @@
 <robot xmlns:xacro="http://www.ros.org/wiki/xacro">
     <xacro:include filename="transmission.xacro"/>
-    <xacro:macro name="leg" params="name mirror mirror_dae front_hind front_hind_dae">
+    <xacro:macro name="leg" params="name mirror mirror_dae front_hind front_hind_dae prefix:='' ">
         <joint name="${name}_hip_joint" type="revolute">
             <xacro:if value="${(mirror_dae == False) and (front_hind_dae == True)}">
@@ -16,5 +16,5 @@
                 <origin rpy="0 0 0" xyz="${-leg_offset_x} ${leg_offset_y} 0"/>
             </xacro:if>
-            <parent link="trunk"/>
+            <parent link="${prefix}trunk"/>
             <child link="${name}_hip"/>
             <axis xyz="1 0 0"/>
@@ -40,5 +40,5 @@
                 <origin rpy="0 0 0" xyz="${-hip_rotor_offset_x} ${hip_rotor_offset_y} 0"/>
             </xacro:if>
-            <parent link="trunk"/>
+            <parent link="${prefix}trunk"/>
             <child link="${name}_hip_rotor"/>
         </joint>
