Commit message: fixed z1 and b2 macro, b2_z1 robot assembled

File: src/b2_description/xacro/b2_robot_macro.urdf.xacro (robot description, xacro)
@@ -152,5 +152,5 @@
                  использовалось в b2_robot).
   ====================================================================== -->
-  <xacro:macro name="b2_ros2_control" params="prefix:=''">
+  <xacro:macro name="b2_ros2_control_list" params="prefix:=''">
     <!-- FL leg -->
     <xacro:joint_control_block name="${prefix}FL_hip_joint"  effort_min="-200" effort_max="200" pos_min="-0.87" pos_max="0.87" init_pos="0.0"/>

File: src/b2_description/xacro/b2_robot_standalone.urdf.xacro (robot description, xacro)
@@ -9,5 +9,5 @@
       <plugin>gz_ros2_control/GazeboSimSystem</plugin>
     </hardware>
-    <xacro:b2_ros2_control prefix=""/>
+    <xacro:b2_ros2_control_list prefix=""/>
   </ros2_control>
   <xacro:include filename="gazebo.xacro"/>

File: src/z1_model/urdf/materials.xacro (robot description, xacro)
@@ -1,7 +1,7 @@
 <?xml version="1.0"?>
 <robot xmlns:xacro="http://www.ros.org/wiki/xacro">
-    <material name="grey">
+    <!-- <material name="grey">
         <color rgba="0.5 0.5 0.5 1.0"/>
-    </material>
+    </material> -->
     <material name="iron_red">
         <color rgba="0.80 0.06 0.06 1.0"/>

File: src/z1_model/urdf/z1_arm_macro.urdf.xacro (robot description, xacro)
@@ -261,5 +261,5 @@
       </link>
       <!-- Нажимной элемент (Finger) -->
-      <link name="z1_Gripper_finger">
+      <link name="${prefix}Gripper_finger">
         <inertial>
             <origin xyz="0.117494 0.0 -0.040887" rpy="0 0 0"/>
@@ -277,5 +277,5 @@
                 <cylinder length="0.036" radius="0.003"/>
             </geometry>
-            <material name="grey"/>
+            <material name="red"/>
         </visual>
         <collision>
@@ -291,15 +291,15 @@
       <!-- Крепление нажимного элемента к статору схвата -->
       <joint name="gripper_stator_to_finger" type="fixed">
-          <parent link="gripperStator"/> <!-- Замените на точное имя link'а вашего статора -->
-          <child link="z1_Gripper_finger"/>
+          <parent link="${prefix}gripperStator"/> <!-- Замените на точное имя link'а вашего статора -->
+          <child link="${prefix}Gripper_finger"/>
           <origin xyz="0 0 0" rpy="0 0 0"/> <!-- Позиции совпадают, как вы указали -->
       </joint>
       <!-- TCP на кончике нажимного элемента -->
       <!-- Пустой линк без массы и визуализации -->
-      <link name="finger_tcp_link"/>
+      <link name="${prefix}finger_tcp_link"/>
       <!-- </link> -->
       <joint name="finger_to_finger_tcp" type="fixed">
-        <parent link="z1_Gripper_finger"/>
-        <child link="finger_tcp_link"/>
+        <parent link="${prefix}Gripper_finger"/>
+        <child link="${prefix}finger_tcp_link"/>
         <!-- Сдвигаем точку ровно туда, где находится край визуального цилиндра -->
         <!-- Цилиндр имеет длину 0.036 и сдвинут на 0.139.
@@ -368,4 +368,15 @@
     </ros2_control>
   </xacro:macro>
+  <xacro:macro name="z1_ros2_control_list" params="prefix:='' use_gripper:=true name:=Z1GazeboSystem">
+    <xacro:joint_controller name="${prefix}joint1" initial_position="0.0"/>
+    <xacro:joint_controller name="${prefix}joint2" initial_position="0.0"/>
+    <xacro:joint_controller name="${prefix}joint3" initial_position="-0.035"/>
+    <xacro:joint_controller name="${prefix}joint4" initial_position="-1.047"/>
+    <xacro:joint_controller name="${prefix}joint5" initial_position="0.0"/>
+    <xacro:joint_controller name="${prefix}joint6" initial_position="0.0"/>
+    <xacro:if value="${use_gripper}">
+      <xacro:joint_controller name="${prefix}jointGripper" initial_position="0.0"/>
+    </xacro:if>
+  </xacro:macro>
   <!-- Локальный макрос-обёртка для регистрации одного джойнта в ros2_control.
        Effort-интерфейс в командах + position/velocity/effort в стейте. -->

File: src/z1_model/urdf/z1_model.urdf.xacro (robot description, xacro)
@@ -271,5 +271,5 @@
                 <cylinder length="0.036" radius="0.003"/>
             </geometry>
-            <material name="grey"/>
+            <material name="red"/>
         </visual>
         <collision>
